Commit message: Adding world link to elbow_flex_motor URDF

File: pr2_component_descriptions/robot_motors/elbow_flex_motor.urdf.xacro (robot description, xacro)
@@ -1,4 +1,5 @@
 <?xml version="1.0"?>
 <robot name="elbow_flex_motor">
+  <link name="world" />
   <joint name="elbow_flex_motor_joint" type="continuous">
     <axis xyz="0 0 1" />
@@ -22,5 +23,4 @@
     <actuator name="r_elbow_flex_motor" />
     <joint name="elbow_flex_motor_joint" />
-    <!-- This is clearly wrong. Need exact number -->
     <mechanicalReduction>${13/3}</mechanicalReduction>
   </transmission>
