Commit message: pr2_component_descriptions tested against new robot_model and new pr2_description

File: pr2_component_descriptions/robot_motors/caster_motor.urdf.xacro (robot description, xacro)
@@ -1,4 +1,5 @@
 <?xml version="1.0"?>
 <robot name="caster_motor">
+  <link name="world" />
   <joint name="caster_motor_joint" type="continuous">
     <axis xyz="0 1 0" />

File: pr2_component_descriptions/robot_motors/forearm_roll_motor.urdf.xacro (robot description, xacro)
@@ -1,4 +1,5 @@
 <?xml version="1.0"?>
 <robot name="r_forearm_roll_motor">
+  <link name="world" />
   <joint name="r_forearm_roll_motor_joint" type="continuous">
     <axis xyz="0 0 1" />

File: pr2_component_descriptions/robot_motors/head_pan_motor.urdf.xacro (robot description, xacro)
@@ -1,4 +1,5 @@
 <?xml version="1.0"?>
 <robot name="head_pan_motor">
+  <link name="world" />
   <joint name="head_pan_motor_joint" type="continuous">
     <axis xyz="0 1 0" />

File: pr2_component_descriptions/robot_motors/head_tilt_motor.urdf.xacro (robot description, xacro)
@@ -1,4 +1,5 @@
 <?xml version="1.0"?>
 <robot name="head_tilt_motor">
+  <link name="world" />
   <joint name="head_tilt_motor_joint" type="continuous">
     <axis xyz="0 1 0" />

File: pr2_component_descriptions/robot_motors/laser_tilt_motor.urdf.xacro (robot description, xacro)
@@ -1,4 +1,5 @@
 <?xml version="1.0"?>
 <robot name="tilting_laser">
+  <link name="world" />
   <joint name="laser_tilt_motor_joint" type="continuous">
     <axis xyz="0 0 1" />

File: pr2_component_descriptions/robot_motors/shoulder_lift_motor.urdf.xacro (robot description, xacro)
@@ -1,4 +1,5 @@
 <?xml version="1.0"?>
 <robot name="shoulder_lift_motor">
+  <link name="world" />
   <joint name="shoulder_lift_motor_joint" type="continuous">
     <axis xyz="0 0 1" />

File: pr2_component_descriptions/robots/gripper.urdf.xacro (robot description, xacro)
@@ -12,4 +12,5 @@
   <include filename="$(find pr2_description)/gazebo/gazebo.urdf.xacro" />
   <xacro:pr2_gripper_v0 side="r" parent="base_link"
+                        reflect="-1.0"
                         screw_reduction="${4.0/1000.0}"
                         gear_ratio="${(729.0/25.0)*(22.0/16.0)}"

File: pr2_component_descriptions/robots/pr2_arm.urdf.xacro (robot description, xacro)
@@ -48,4 +48,5 @@
   </xacro:pr2_forearm_v0>
   <xacro:pr2_gripper_v0 side="r" parent="r_wrist_roll_link"
+                        reflect="-1.0"
                screw_reduction="${4.0/1000.0}"
                gear_ratio="${(729.0/25.0)*(22.0/16.0)}"

File: pr2_component_descriptions/robots/pr2_left_arm.urdf.xacro (robot description, xacro)
@@ -48,4 +48,5 @@
   </xacro:pr2_forearm_v0>
   <xacro:pr2_gripper_v0 side="l" parent="l_wrist_roll_link"
+                        reflect="1.0"
                screw_reduction="${4.0/1000.0}"
                gear_ratio="${(729.0/25.0)*(22.0/16.0)}"
