Commit message: Moved all URDF files out of qualification to pr2_component_descriptions. #4465

File: pr2_component_descriptions/robot_motors/gripper_motor.urdf.xacro (robot description, xacro)
@@ -1,4 +1,5 @@
 <?xml version="1.0"?>
 <robot name="gripper_motor">
+  <link name="world" />
   <joint name="gripper_motor_joint" type="prismatic" >
     <axis xyz="0 1 0" />
