Commit message: With Stu's help got experimetal laser tilt running smoothly

File: life_test/laser_tilt_test_2/laser_tilt_2.urdf (robot description, URDF)
Before this commit: robot tilting_laser, 3 links, 2 joints
Joints:
- joint laser_tilt_mount_joint: limit lower=-0.7854 upper=1.48353 effort=0.65 velocity=10.0 -> lower=-0.7 upper=1.6 effort=10000 velocity=1000000.0
